File: TinyGS_PCB/test_project/test_project.kicad_pcb (KiCad board)
At the start: 2 copper layers, 45.7 x 119.4 mm, 6 parts, among them J1 Power Input, U1 ESP32, U2 E32400M30S, U3 OLED

Commit message: fixed mistakes on pcb and software
Connections:
- U1 pad 6: Net-(R1-Pad2) -> Net-(R2-Pad2)
- U1 pad 7: Net-(R2-Pad2) -> Net-(R1-Pad2)
Routing:
- net Net-(R2-Pad2): track 20.3 -> 40.0 mm
- net Net-(R1-Pad2): track 10.6 -> 12.5 mm
Changed lines of the file:
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@@
       (net 11 "unconnected-(U1-Pad5)") (pinfunction "GPIO35") (pintype "bidirectional"))
     (pad "6" thru_hole oval (at 1.55 18.72 180) (size 1.7 1.7) (drill 1) (layers *.Cu *.Mask)
-      (net 4 "Net-(R1-Pad2)") (pinfunction "GPIO32") (pintype "bidirectional"))
+      (net 6 "Net-(R2-Pad2)") (pinfunction "GPIO32") (pintype "bidirectional"))
     (pad "7" thru_hole oval (at 1.55 21.26 180) (size 1.7 1.7) (drill 1) (layers *.Cu *.Mask)
-      (net 6 "Net-(R2-Pad2)") (pinfunction "GPIO33") (pintype "bidirectional"))
+      (net 4 "Net-(R1-Pad2)") (pinfunction "GPIO33") (pintype "bidirectional"))
     (pad "8" thru_hole oval (at 1.55 23.8 180) (size 1.7 1.7) (drill 1) (layers *.Cu *.Mask)
       (net 12 "unconnected-(U1-Pad8)") (pinfunction "GPIO25") (pintype "bidirectional"))
@@
   (segment (start 144.78 53.34) (end 134.62 53.34) (width 0.25) (layer "B.Cu") (net 3))
   (segment (start 144.78 91.44) (end 147.32 88.9) (width 0.25) (layer "B.Cu") (net 3))
-  (segment (start 139.7 96.52) (end 139.7 101.6) (width 0.25) (layer "F.Cu") (net 4))
-  (segment (start 134.5075 95.7925) (end 138.9725 95.7925) (width 0.25) (layer "F.Cu") (net 4))
-  (segment (start 138.9725 95.7925) (end 139.7 96.52) (width 0.25) (layer "F.Cu") (net 4))
+  (segment (start 137.9565 93.2525) (end 134.5075 93.2525) (width 0.25) (layer "F.Cu") (net 4))
+  (segment (start 139.7 94.996) (end 137.9565 93.2525) (width 0.25) (layer "F.Cu") (net 4))
+  (segment (start 139.7 101.6) (end 139.7 94.996) (width 0.25) (layer "F.Cu") (net 4))
   (segment (start 130.884 59.764) (end 130.884 57.72) (width 0.25) (layer "F.Cu") (net 5))
   (segment (start 137.16 63.5) (end 134.62 60.96) (width 0.25) (layer "F.Cu") (net 5))
@@
   (segment (start 132.08 60.96) (end 130.884 59.764) (width 0.25) (layer "F.Cu") (net 5))
   (segment (start 137.16 73.66) (end 137.16 63.5) (width 0.25) (layer "F.Cu") (net 5))
-  (segment (start 136.4325 93.2525) (end 134.5075 93.2525) (width 0.25) (layer "F.Cu") (net 6))
   (segment (start 139.7 86.36) (end 142.24 86.36) (width 0.25) (layer "F.Cu") (net 6))
-  (segment (start 137.16 93.98) (end 136.4325 93.2525) (width 0.25) (layer "F.Cu") (net 6))
-  (segment (start 144.78 88.9) (end 144.78 91.44) (width 0.25) (layer "F.Cu") (net 6))
-  (segment (start 142.24 93.98) (end 137.16 93.98) (width 0.25) (layer "F.Cu") (net 6))
-  (segment (start 144.78 91.44) (end 142.24 93.98) (width 0.25) (layer "F.Cu") (net 6))
+  (segment (start 139.192 105.156) (end 137.414 103.378) (width 0.25) (layer "F.Cu") (net 6))
+  (segment (start 144.78 88.9) (end 144.78 104.648) (width 0.25) (layer "F.Cu") (net 6))
+  (segment (start 136.1785 95.7925) (end 134.5075 95.7925) (width 0.25) (layer "F.Cu") (net 6))
+  (segment (start 144.78 104.648) (end 144.272 105.156) (width 0.25) (layer "F.Cu") (net 6))
+  (segment (start 137.414 97.028) (end 136.1785 95.7925) (width 0.25) (layer "F.Cu") (net 6))
+  (segment (start 137.414 103.378) (end 137.414 97.028) (width 0.25) (layer "F.Cu") (net 6))
+  (segment (start 144.272 105.156) (end 139.192 105.156) (width 0.25) (layer "F.Cu") (net 6))
   (segment (start 142.24 86.36) (end 144.78 88.9) (width 0.25) (layer "F.Cu") (net 6))
   (segment (start 121.9545 88.1725) (end 134.5075 88.1725) (width 0.25) (layer "F.Cu") (net 13))
